File: hardware/bd0/bd0.kicad_sch (KiCad schematic)
At the start: 3 parts, among them J1 USB_C_Receptacle_USB2.0, J2 SJ-43514, U1 ATSAMD21G15B-A

Commit message: Finished BD0 schematic and routing
Parts:
- removed J2: SJ-43514, Conn_CUI_SJ-4351:CUI-SJ-43514-0, symbol eec:SJ-43514
- added C1, C8, C9: 1uF, Capacitor_SMD:C_0603_1608Metric, symbol Device:C
- added C2, C3, C4, C5: 0.1uF, Capacitor_SMD:C_0603_1608Metric, symbol Device:C
- added C6, C7: 10uF, Capacitor_SMD:C_0603_1608Metric, symbol Device:C
- added D1, D2, D3: LED, Diode_SMD:D_0603_1608Metric, symbol Device:LED
- added FB1: FerriteBead, Inductor_SMD:L_0603_1608Metric, symbol Device:FerriteBead
- added J1: Conn_02x03_Odd_Even, Connector:Tag-Connect_TC2030-IDC-NL_2x03_P1.27mm_Vertical, symbol Connector_Generic:Conn_02x03_Odd_Even
- added J20: USB_C_Receptacle_USB2.0, Connector_USB:USB_C_Receptacle_JAE_DX07S016JA1R1500, symbol Connector:USB_C_Receptacle_USB2.0
- added J3, J30: SJ-43514, Conn_CUI_SJ-4351:CUI-SJ-43514-SMT-0, symbol Conn_CUI_SJ-4351:SJ-43514
- added R1, R3, R4: 10k, Resistor_SMD:R_0603_1608Metric, symbol Device:R_US
- added R2: 1k, Resistor_SMD:R_0603_1608Metric, symbol Device:R_US
- added R5, R6, R7: 470, Resistor_SMD:R_0603_1608Metric, symbol Device:R_US
- added U2: AP2127N-3.3, Package_TO_SOT_SMD:SOT-23, symbol Regulator_Linear:AP2127N-3.3
- renumbered J1 to J2
Connections:
- net +3V3: now also U1.17 (VDDIO), U1.36 (VDDIO), U1.44 (VDDIN), C3.1, C4.1, C5.1, C6.1, C9.1, FB1.1, J1.1 (Pin_1), J3.2 (Tip), J30.2 (Tip), R1.1, R2.1, R3.1, R4.1, U2.2 (VO)
- net GND: now also C1.2, C2.2, C3.2, C4.2, C5.2, C6.2, C7.2, C8.2, C9.2, J1.5 (Pin_5), J20.A1 (GND), J20.A12 (GND), J20.B1 (GND), J20.B12 (GND), J20.S1 (SHIELD), J3.1 (Sleeve), J30.1 (Sleeve), R5.2, R6.2, R7.2, U2.1 (GND)
- net USB_DP: now also J20.A6 (D+), J20.B6 (D+)
- net home_thumb: now also U1.25 (PA16); no longer U1.13 (PA08)
- net +5V: now reaches J2.A4 (VBUS), J2.A9 (VBUS), J2.B4 (VBUS), J2.B9 (VBUS)
- net +5V: now also C8.1, J20.A4 (VBUS), J20.A9 (VBUS), J20.B4 (VBUS), J20.B9 (VBUS), U2.3 (VI)
- net middle_top: now reaches U1.10 (PA05)
- net ring_bottom: now reaches U1.11 (PA06)
- net ring_home: now reaches U1.12 (PA07)
- net ring_top: now reaches U1.14 (PA09)
- net pinky_bottom: now reaches U1.15 (PA10)
- net pinky_home: now reaches U1.16 (PA11)
- net index_home: now reaches U1.2 (PA01)
- net pinky_top: now reaches U1.21 (PA12)
- net outer_bottom: now reaches U1.22 (PA13)
- net outer_home: now reaches U1.23 (PA14)
- net outer_top: now reaches U1.24 (PA15)
- net far_thumb: now reaches U1.26 (PA17)
- net inner_bottom: now reaches U1.27 (PA18)
- net inner_home: now reaches U1.28 (PA19)
- net inner_top: now reaches U1.29 (PA20)
- net index_top: now reaches U1.3 (PA02)
- net SCL: now reaches U1.32 (PA23)
- net SCL: now also J3.4 (Ring2), J30.4 (Ring2), R4.2
- net LED0: now reaches U1.37 (PB22)
- net LED0: now also D1.1 (K)
- net LED1: now reaches U1.38 (PB23)
- net LED1: now also D2.1 (K)
- net LED2: now reaches U1.39 (PA27)
- net LED2: now also D3.1 (K)
- net middle_bottom: now reaches U1.4 (PA03)
- net RESETn: now reaches U1.40 (~{RESET})
- net RESETn: now also J1.3 (Pin_3), R1.2
- net index_bottom: now reaches U1.41 (PA28)
- net +1V2: now reaches U1.43 (VDDCORE)
- net +1V2: now also C1.1
- net SWCLK: now reaches U1.45 (PA30)
- net SWCLK: now also J1.4 (Pin_4), R2.2
- net SWDIO: now reaches U1.46 (PA31)
- net SWDIO: now also J1.2 (Pin_2)
- net 3V3A: now reaches U1.6 (VDDANA)
- net 3V3A: now also C2.1, C7.1, FB1.2
- net middle_home: now reaches U1.9 (PA04)
- net RX: no longer names the net of U1.30 (PA21)
- net TX renamed SDA
- net SDA: now also J3.3 (Ring1), J30.3 (Ring1), R3.2
- net USB_DM renamed USB_DN
- net USB_DN: now also J20.A7 (D-), J20.B7 (D-)
- new net: D2.2 (A), R6.1
- new net: D3.2 (A), R7.1
- new net: D1.2 (A), R5.1
- new net near_thumb: U1.13 (PA08)
- no-connect marks 4 -> 16
Other:
- moved on the sheet: J2, U1
